File: KayproKeyboard.kicad_pcb (KiCad board)
At the start: 2 copper layers, 427.9 x 155 mm, 163 parts, among them J1 Conn_01x06_Pin, J2 Conn_01x06, J3 Conn_01x06, SW1 A_Key, SW10 J_Key, SW11 K_Key, SW12 L_Key, SW13 M_Key, SW14 N_Key, SW15 O_Key, SW16 P_Key, SW17 Q_Key, SW18 R_Key, SW19 S_Key, SW2 B_Key, SW20 T_Key, SW21 U_Key, SW22 V_Key, SW23 W_Key, SW24 X_Key, SW25 Y_Key, SW26 Z_Key, SW27 1_Key, SW28 2_Key, SW29 3_Key, SW3 C_Key, SW30 4_Key, SW31 5_Key, SW32 6_Key, SW33 7_Key, SW34 8_Key, SW35 9_Key, SW36 0_Key, SW37 -_Key, SW38 =_Key, SW39 `_Key, SW4 D_Key, SW40 ;_Key, SW41 '_Key, SW42 \_Key, SW43 ,_Key, SW44 ._Key, SW45 /_Key, SW46 LSHIFT_Key, SW47 RSHIFT_Key, SW49 CTRL_Key, SW5 E_Key, SW50 CAPS_Key, SW51 DEL_Key, SW52 BACKSPACE_Key, SW53 SPACE_Key, SW54 ESC_Key, SW55 TAB_Key, SW56 RETURN_Key, SW57 LINEFEED_Key, SW58 UP_Key, SW59 DOWN_Key, SW6 F_Key, SW60 LEFT_Key, SW61 RIGHT_Key, SW62 NUM0_Key, SW63 NUM1_Key, SW64 NUM2_Key, SW65 NUM3_Key, SW66 NUM4_Key, SW67 NUM5_Key, SW68 NUM6_Key, SW69 NUM7_Key, SW7 G_Key, SW70 NUM8_Key, SW71 NUM9_Key, SW72 NUM._Key, SW73 NUMENTER_Key, SW74 NUM-_Key, SW75 NUM,_Key, SW76 [_KEY, SW77 ]_KEY, SW8 H_Key, SW9 I_Key, U1 Pico

Commit message: Add files via upload
Connections:
- J2 pad 3: GND -> +3.3V
- J2 pad 4: +3.3V -> GND
Routing:
- net Net-(D60-A): track 0.00 -> 68.1 mm, vias 0 -> 3
- net Net-(D62-A): track 0.00 -> 22.9 mm
- net Net-(D63-A): track 0.00 -> 18.0 mm
- net Net-(D61-A): track 0.00 -> 17.8 mm
- net +3.3V: track 158.3 -> 160.5 mm
- net GND: track 366.0 -> 366.6 mm
- removed copper zone on B.Cu, net (none)
- removed copper zone on F.Cu, net (none)
Changed lines of the file:
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@@
 			(keep_end_layers yes)
 			(zone_layer_connections)
-			(net "GND")
+			(net "+3.3V")
 			(pinfunction "Pin_3_3")
 			(pintype "passive")
@@
 			(keep_end_layers yes)
 			(zone_layer_connections)
-			(net "+3.3V")
+			(net "GND")
 			(pinfunction "Pin_4_4")
 			(pintype "passive")
@@
 	)
 	(image
-		(at 154.77 32.52)
+		(at 156.125001 33.25)
 		(layer "F.SilkS")
-		(scale 0.0625351)
+		(scale 0.0646178)
 		(data "iVBORw0KGgoAAAANSUhEUgAABXkAAAXBCAYAAADIDJy0AAAACXBIWXMAABYlAAAWJQFJUiTwAAAg"
 			"AElEQVR4nOzd4XUb17U24NdZ9z/RgeAKRFcgqAIxFQSuQHQFpiuIXEGgCkJVEKqCkBWE7ICoQN+P"
@@
 	)
 	(segment
+		(start 402.76 60.21)
+		(end 406.85 56.12)
+		(width 0.5)
+		(layer "F.Cu")
+		(net "Net-(D62-A)")
+	)
+	(segment
+		(start 414.025 65.675)
+		(end 416.1 67.75)
+		(width 0.5)
+		(layer "F.Cu")
+		(net "Net-(D62-A)")
+	)
+	(segment
+		(start 409.752032 56.12)
+		(end 414.025 60.392968)
+		(width 0.5)
+		(layer "F.Cu")
+		(net "Net-(D62-A)")
+	)
+	(segment
+		(start 414.025 60.392968)
+		(end 414.025 65.675)
+		(width 0.5)
+		(layer "F.Cu")
+		(net "Net-(D62-A)")
+	)
+	(segment
+		(start 406.85 56.12)
+		(end 409.752032 56.12)
+		(width 0.5)
+		(layer "F.Cu")
+		(net "Net-(D62-A)")
+	)
+	(segment
 		(start 321.24 121.283866)
 		(end 321.24 125.03)
@@
 	)
 	(segment
-		(start 340.89 33.67)
-		(end 340.89 49.6)
-		(width 1)
+		(start 170.35 108.41)
+		(end 164.61 108.41)
+		(width 0.5)
 		(layer "F.Cu")
 		(net "GND")
 	)
 	(segment
-		(start 187.62 53.56)
-		(end 185.08 56.1)
-		(width 0.5)
+		(start 340.89 33.67)
+		(end 340.89 49.6)
+		(width 1)
 		(layer "F.Cu")
 		(net "GND")
 	)
 	(segment
-		(start 170.35 108.41)
-		(end 164.61 108.41)
+		(start 175.17 113.23)
+		(end 170.35 108.41)
 		(width 0.5)
 		(layer "F.Cu")
@@
 	)
 	(segment
+		(start 187.585 52.41)
+		(end 187.62 52.375)
+		(width 0.5)
+		(layer "F.Cu")
+		(net "GND")
+	)
+	(segment
 		(start 248.95 48.63)
 		(end 251.83 45.75)
@@
 	)
 	(segment
-		(start 187.62 46)
-		(end 187.62 53.56)
+		(start 167.42 52.41)
+		(end 187.585 52.41)
 		(width 0.5)
 		(layer "F.Cu")
@@
 	)
 	(segment
+		(start 187.62 56.1)
+		(end 187.62 52.375)
+		(width 0.5)
+		(layer "F.Cu")
+		(net "GND")
+	)
+	(segment
 		(start 258.13 37.88)
 		(end 266.25 46)
@@
 	)
 	(segment
-		(start 266 45.75)
-		(end 266.25 46)
-		(width 1)
+		(start 163.26 107.06)
+		(end 163.26 56.57)
+		(width 0.5)
 		(layer "F.Cu")
 		(net "GND")
 	)
 	(segment
-		(start 175.17 113.23)
-		(end 170.35 108.41)
+		(start 187.62 52.375)
+		(end 187.62 46)
 		(width 0.5)
 		(layer "F.Cu")
@@
 	)
 	(segment
+		(start 266 45.75)
+		(end 266.25 46)
+		(width 1)
+		(layer "F.Cu")
+		(net "GND")
+	)
+	(segment
 		(start 258.13 31.7)
 		(end 258.13 37.88)
@@
 	)
 	(segment
+		(start 164.61 108.41)
+		(end 163.26 107.06)
+		(width 0.5)
+		(layer "F.Cu")
+		(net "GND")
+	)
+	(segment
 		(start 315.49 34.33)
 		(end 315.49 49.6)
@@
 	)
 	(segment
-		(start 163.26 107.06)
-		(end 163.26 56.57)
-		(width 0.5)
-		(layer "F.Cu")
-		(net "GND")
-	)
-	(segment
-		(start 167.42 52.41)
-		(end 181.39 52.41)
-		(width 0.5)
-		(layer "F.Cu")
-		(net "GND")
-	)
-	(segment
 		(start 299.35 34.95)
 		(end 314.92 34.95)
@@
 	)
 	(segment
-		(start 164.61 108.41)
-		(end 163.26 107.06)
-		(width 0.5)
-		(layer "F.Cu")
-		(net "GND")
-	)
-	(segment
 		(start 315.49 34.33)
 		(end 328.28 34.33)
@@
 	)
 	(segment
-		(start 181.39 52.41)
-		(end 185.08 56.1)
-		(width 0.5)
-		(layer "F.Cu")
-		(net "GND")
-	)
-	(segment
 		(start 353.59 32.72)
 		(end 353.59 31.82)
@@
 		(width 0.5)
 		(layer "B.Cu")
-		(net "+3.3V")
+		(net "GND")
 	)
 	(segment
 		(start 248.7 40.87)
-		(end 263.62 40.87)
+		(end 240.71 48.86)
 		(width 0.5)
 		(layer "B.Cu")
@@
 	)
 	(segment
-		(start 240.71 48.86)
+		(start 263.62 40.87)
 		(end 248.7 40.87)
 		(width 0.5)
@@
 	)
 	(segment
-		(start 320.57 31.82)
-		(end 311.26 22.51)
-		(width 1)
+		(start 192.32 48.86)
+		(end 185.08 56.1)
+		(width 0.5)
 		(layer "B.Cu")
 		(net "+3.3V")
 	)
 	(segment
-		(start 263.62 40.87)
-		(end 266.25 43.5)
+		(start 240.71 48.86)
+		(end 192.32 48.86)
 		(width 0.5)
 		(layer "B.Cu")
@@
 	)
 	(segment
-		(start 311.26 22.51)
-		(end 278.66 22.51)
+		(start 320.57 31.82)
+		(end 311.26 22.51)
 		(width 1)
 		(layer "B.Cu")
@@
 	)
 	(segment
-		(start 194.25 48.86)
-		(end 240.71 48.86)
-		(width 0.5)
+		(start 311.26 22.51)
+		(end 278.66 22.51)
+		(width 1)
 		(layer "B.Cu")
 		(net "+3.3V")
 	)
 	(segment
-		(start 187.62 55.49)
-		(end 194.25 48.86)
+		(start 266.25 43.5)
+		(end 263.62 40.87)
 		(width 0.5)
 		(layer "B.Cu")
@@
 	)
 	(segment
+		(start 383.71 60.21)
+		(end 385.02 61.52)
+		(width 0.5)
+		(layer "F.Cu")
+		(net "Net-(D63-A)")
+	)
+	(segment
+		(start 388.984466 67.75)
+		(end 397.25 67.75)
+		(width 0.5)
+		(layer "F.Cu")
+		(net "Net-(D63-A)")
+	)
+	(segment
+		(start 385.02 61.52)
+		(end 385.02 63.785534)
+		(width 0.5)
+		(layer "F.Cu")
+		(net "Net-(D63-A)")
+	)
+	(segment
+		(start 385.02 63.785534)
+		(end 388.984466 67.75)
+		(width 0.5)
+		(layer "F.Cu")
+		(net "Net-(D63-A)")
+	)
+	(segment
 		(start 288.45 159.284366)
 		(end 288.45 163.59)
@@
 	)
 	(segment
+		(start 377.87 67.75)
+		(end 380.27 70.15)
+		(width 0.5)
+		(layer "F.Cu")
+		(net "Net-(D60-A)")
+	)
+	(segment
+		(start 405.275 70.15)
+		(end 407.175 68.25)
+		(width 0.5)
+		(layer "F.Cu")
+		(net "Net-(D60-A)")
+	)
+	(segment
+		(start 380.27 70.15)
+		(end 405.275 70.15)
+		(width 0.5)
+		(layer "F.Cu")
+		(net "Net-(D60-A)")
+	)
+	(segment
+		(start 426.525 65.925)
+		(end 431.4 65.925)
+		(width 0.5)
+		(layer "F.Cu")
+		(net "Net-(D60-A)")
+	)
+	(segment
+		(start 431.4 65.925)
+		(end 432.4 64.925)
+		(width 0.5)
+		(layer "F.Cu")
+		(net "Net-(D60-A)")
+	)
+	(via
+		(at 432.4 64.925)
+		(size 0.6)
+		(drill 0.3)
+		(layers "F.Cu" "B.Cu")
+		(net "Net-(D60-A)")
+	)
+	(via
+		(at 407.175 68.25)
+		(size 0.6)
+		(drill 0.3)
+		(layers "F.Cu" "B.Cu")
+		(net "Net-(D60-A)")
+	)
+	(via
+		(at 426.525 65.925)
+		(size 0.6)
+		(drill 0.3)
+		(layers "F.Cu" "B.Cu")
+		(net "Net-(D60-A)")
+	)
+	(segment
+		(start 432.4 64.925)
+		(end 437.115 60.21)
+		(width 0.5)
+		(layer "B.Cu")
+		(net "Net-(D60-A)")
+	)
+	(segment
+		(start 409.5 65.925)
+		(end 426.525 65.925)
+		(width 0.5)
+		(layer "B.Cu")
+		(net "Net-(D60-A)")
+	)
+	(segment
+		(start 407.175 68.25)
+		(end 409.5 65.925)
+		(width 0.5)
+		(layer "B.Cu")
+		(net "Net-(D60-A)")
+	)
+	(segment
+		(start 437.115 60.21)
+		(end 440.86 60.21)
+		(width 0.5)
+		(layer "B.Cu")
+		(net "Net-(D60-A)")
+	)
+	(segment
 		(start 261.1 27.05)
 		(end 265.75 31.7)
@@
 	)
 	(segment
+		(start 430.069188 60.21)
+		(end 434.94 65.080812)
+		(width 0.5)
+		(layer "F.Cu")
+		(net "Net-(D61-A)")
+	)
+	(segment
+		(start 421.81 60.21)
+		(end 430.069188 60.21)
+		(width 0.5)
+		(layer "F.Cu")
+		(net "Net-(D61-A)")
+	)
+	(segment
+		(start 434.94 65.080812)
+		(end 434.94 67.75)
+		(width 0.5)
+		(layer "F.Cu")
+		(net "Net-(D61-A)")
+	)
+	(segment
 		(start 363.250366 117.4175)
 		(end 359.24 121.427866)
@@
 		(polygon
 			(pts
-				(xy 144.73 173.75) (xy 144.73 21.62) (xy 569.63 21.62) (xy 569.63 173.75)
-			)
-		)
-	)
-	(zone
-		(layers "F.Cu" "B.Cu")
-		(name "BLANK")
-		(hatch edge 0.5)
-		(priority 1)
-		(connect_pads
-			(clearance 0.5)
-		)
-		(min_thickness 0.25)
-		(fill yes
-			(thermal_gap 0.5)
-			(thermal_bridge_width 0.5)
-			(island_removal_mode 1)
-		)
-		(polygon
-			(pts
-				(xy 150.25 23.88) (xy 150.25 167.96) (xy 565.85 167.96) (xy 565.85 23.89) (xy 565.81 23.89) (xy 565.81 24.2)
-				(xy 565.81 23.88)
+				(xy 570.475 20.525) (xy 143.975 20.525) (xy 143.975 174.2) (xy 570.475 174.2)
 			)
 		)
