File: KayproKeyboard.kicad_sch (KiCad schematic)
At the start: 163 parts, among them J1 Conn_01x06_Pin, J2 Conn_01x06, J3 Conn_01x06, SW1 A_Key, SW10 J_Key, SW11 K_Key, SW12 L_Key, SW13 M_Key, SW14 N_Key, SW15 O_Key, SW16 P_Key, SW17 Q_Key, SW18 R_Key, SW19 S_Key, SW2 B_Key, SW20 T_Key, SW21 U_Key, SW22 V_Key, SW23 W_Key, SW24 X_Key, SW25 Y_Key, SW26 Z_Key, SW27 1_Key, SW28 2_Key, SW29 3_Key, SW3 C_Key, SW30 4_Key, SW31 5_Key, SW32 6_Key, SW33 7_Key, SW34 8_Key, SW35 9_Key, SW36 0_Key, SW37 -_Key, SW38 =_Key, SW39 `_Key, SW4 D_Key, SW40 ;_Key, SW41 '_Key, SW42 \_Key, SW43 ,_Key, SW44 ._Key, SW45 /_Key, SW46 LSHIFT_Key, SW47 RSHIFT_Key, SW49 CTRL_Key, SW5 E_Key, SW50 CAPS_Key, SW51 DEL_Key, SW52 BACKSPACE_Key, SW53 SPACE_Key, SW54 ESC_Key, SW55 TAB_Key, SW56 RETURN_Key, SW57 LINEFEED_Key, SW58 UP_Key, SW59 DOWN_Key, SW6 F_Key, SW60 LEFT_Key, SW61 RIGHT_Key, SW62 NUM0_Key, SW63 NUM1_Key, SW64 NUM2_Key, SW65 NUM3_Key, SW66 NUM4_Key, SW67 NUM5_Key, SW68 NUM6_Key, SW69 NUM7_Key, SW7 G_Key, SW70 NUM8_Key, SW71 NUM9_Key, SW72 NUM._Key, SW73 NUMENTER_Key, SW74 NUM-_Key, SW75 NUM,_Key, SW76 [_KEY, SW77 ]_KEY, SW8 H_Key, SW9 I_Key, U1 Pico

Commit message: Add files via upload
Connections:
- net +3.3V: now also J2.3 (Pin_3); no longer J2.4 (Pin_4)
- net GND: now also J2.4 (Pin_4); no longer J2.3 (Pin_3)
Changed lines of the file:
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@@
 	(wire
 		(pts
-			(xy 200.66 40.64) (xy 204.47 40.64)
-		)
-		(stroke
-			(width 0)
-			(type default)
-		)
-	)
-	(wire
-		(pts
 			(xy 128.27 25.4) (xy 129.54 25.4)
 		)
@@
 	(wire
 		(pts
+			(xy 200.66 40.64) (xy 204.47 40.64)
+		)
+		(stroke
+			(width 0)
+			(type default)
+		)
+	)
+	(wire
+		(pts
 			(xy 85.09 140.97) (xy 87.63 140.97)
 		)
@@
 	(wire
 		(pts
+			(xy 200.66 38.1) (xy 204.47 38.1)
+		)
+		(stroke
+			(width 0)
+			(type default)
+		)
+	)
+	(wire
+		(pts
 			(xy 31.75 64.77) (xy 35.56 64.77)
 		)
@@
 	(wire
 		(pts
-			(xy 200.66 38.1) (xy 204.47 38.1)
-		)
-		(stroke
-			(width 0)
-			(type default)
-		)
-	)
-	(wire
-		(pts
 			(xy 135.89 148.59) (xy 135.89 149.86)
 		)
@@
 	(symbol
 		(lib_id "power:GND")
-		(at 200.66 40.64 270)
+		(at 200.66 38.1 270)
 		(unit 1)
 		(body_style 1)
@@
 		(fields_autoplaced yes)
 		(property "Reference" "#PWR023"
-			(at 194.31 40.64 0)
+			(at 194.31 38.1 0)
 			(hide yes)
 			(show_name no)
@@
 		)
 		(property "Value" "GND"
-			(at 196.85 40.6399 90)
+			(at 196.85 38.0999 90)
 			(show_name no)
 			(do_not_autoplace no)
@@
 		)
 		(property "Footprint" ""
-			(at 200.66 40.64 0)
+			(at 200.66 38.1 0)
 			(hide yes)
 			(show_name no)
@@
 		)
 		(property "Datasheet" ""
-			(at 200.66 40.64 0)
+			(at 200.66 38.1 0)
 			(hide yes)
 			(show_name no)
@@
 		)
 		(property "Description" "Power symbol creates a global label with name \"GND\" , ground"
-			(at 200.66 40.64 0)
+			(at 200.66 38.1 0)
 			(hide yes)
 			(show_name no)
@@
 	(symbol
 		(lib_id "power:+3.3V")
-		(at 200.66 38.1 90)
+		(at 200.66 40.64 90)
 		(unit 1)
 		(body_style 1)
@@
 		(fields_autoplaced yes)
 		(property "Reference" "#PWR024"
-			(at 204.47 38.1 0)
+			(at 204.47 40.64 0)
 			(hide yes)
 			(show_name no)
@@
 		)
 		(property "Value" "+3.3V"
-			(at 196.85 38.0999 90)
+			(at 196.85 40.6399 90)
 			(show_name no)
 			(do_not_autoplace no)
@@
 		)
 		(property "Footprint" ""
-			(at 200.66 38.1 0)
+			(at 200.66 40.64 0)
 			(hide yes)
 			(show_name no)
@@
 		)
 		(property "Datasheet" ""
-			(at 200.66 38.1 0)
+			(at 200.66 40.64 0)
 			(hide yes)
 			(show_name no)
@@
 		)
 		(property "Description" "Power symbol creates a global label with name \"+3.3V\""
-			(at 200.66 38.1 0)
+			(at 200.66 40.64 0)
 			(hide yes)
 			(show_name no)
